File: main_board4.sch (KiCad schematic (older format))
At the start: 263 parts

Commit message: update sche
Parts:
- added D? (x15): DIODE, Diode_SMD:D_MiniMELF, symbol lee_mech_key_comp:DIODE
- added DEC, DEL, DEV, END, INS, MUL, No2, No3, No5, No6, No8, No9, PLUS, R_Enter, R_minus: SWITCH_PUSH, sw_fprint_wLed:CHERRY_PCB_100H, symbol lee_mech_key_comp:SWITCH_PUSH
- added R? (x15): R, Resistor_SMD:R_0805_2012Metric, symbol lee_mech_key_comp:R
- renumbered RCTRL1 to DOWN1, DELETE1 to HOME1, RALT1 to MENU1, RIGHT1 to NO0, END1 to NO1, PAGEDOWN1 to NO4, PAGEUP1 to NO7, HOME1 to NUMLOCK, PRINTSCREEN1 to PAUSE1, INSERT1 to PRSCREEN1, DOWN1 to RIGHT1
Connections:
- net labels added: LED_C1, LED_C2, LED_C3, Row_1, Row_2, Row_3, Row_4, Row_5, Row_6
- wire segments 746 -> 830
Other:
- note added: "Col-10\n"
- note added: "Col-11"
- note added: "Col-12"
- note added: "Col-13"
- note added: "Col-14"
- note added: "Col-15"
- note added: "Col-16"
- note added: "Col-17"
- note added: "Col-2"
- note added: "Col-3\n"
- note added: "Col-4"
- note added: "Col-5"
- note added: "Col-6"
- note added: "Col-7\n"
- note added: "Col-8"
- note added: "Col-9"
- note added: "Col_1\n"

Commit message: update wiring
Connections:
- wire segments 830 -> 829
Changed lines of the file:
@@
 EESchema Schematic File Version 4
 LIBS:power
-LIBS:device
 LIBS:74xx
-LIBS:audio
-LIBS:interface
 LIBS:main_board4-cache
 EELAYER 26 0
 EELAYER END
-$Descr A2 23386 16535
+$Descr A1 33110 23386
 encoding utf-8
 Sheet 1 1
-Title ""
-Date ""
-Rev ""
+Title "mechkey_mainboard_v2"
+Date "2018-11-13"
+Rev "3"
 Comp ""
 Comment1 ""
@@
 	4600 6600 5650 6600
 Wire Wire Line
-	23300 10850 16650 10850
-Wire Wire Line
 	15950 10850 15950 11050
 Wire Wire Line
@@
 Wire Wire Line
 	4600 7200 5650 7200
-Connection ~ 23300 7200
 Wire Wire Line
 	4600 7650 4600 7800
@@
 	4600 7800 5650 7800
 Wire Wire Line
-	13100 10700 13100 11250
-Wire Wire Line
-	11800 11000 11800 10450
-Wire Wire Line
-	11800 10450 13950 10450
-Wire Wire Line
 	4600 9050 4600 8900
 Wire Wire Line
@@
 Wire Wire Line
 	4600 9650 5650 9650
-Connection ~ 23200 9650
 Wire Wire Line
 	4600 8300 4600 8500
 Wire Wire Line
 	4600 8500 5650 8500
-Connection ~ 23250 8500
 Wire Wire Line
 	5650 6450 5650 6600
@@
 Wire Wire Line
 	13950 10450 13950 10300
-Connection ~ 13950 10450
 Wire Wire Line
 	14000 10950 14000 10700
@@
 $EndComp
 Wire Wire Line
-	23300 7200 23300 10850
-Wire Wire Line
-	23200 9650 23200 9050
-Wire Wire Line
 	5650 6600 6700 6600
 Wire Wire Line
@@
 Wire Wire Line
 	16650 10850 15950 10850
-Wire Wire Line
-	14000 10700 13100 10700
 $Comp
 L lee_mech_key_comp:R R7
@@
 	17350 7300 16300 7300
 Wire Wire Line
-	19150 5700 19150 6300
+	19150 5650 19150 6300
 Wire Wire Line
-	18100 5650 18100 6300
+	18100 5600 18100 6300
 Wire Wire Line
-	17050 5600 17050 6300
+	17050 5550 17050 6300
 Wire Wire Line
-	16000 5550 16000 6300
+	16000 5500 16000 6300
 Wire Wire Line
 	14950 5450 14950 6300
@@
 	18250 9200 19300 9200
 Wire Wire Line
-	23600 7900 23600 6800
-Wire Wire Line
-	23350 8550 23350 8100
-Wire Wire Line
-	23400 8150 23400 9150
-Wire Wire Line
-	23450 8200 23450 9750
-Wire Wire Line
 	7850 14450 7850 14700
 Wire Wire Line
@@
 	8550 14900 23700 14900
 Wire Wire Line
-	23650 6800 23650 14850
+	23650 7900 23650 14850
 Wire Wire Line
 	23650 14850 8600 14850
@@
 	8600 13200 23600 13200
 Wire Wire Line
-	23600 13200 23600 8100
+	23600 13200 23600 8550
 Wire Wire Line
-	23550 8150 23550 13150
+	23550 9150 23550 13150
 Wire Wire Line
 	23550 13150 8550 13150
@@
 	8500 13100 23500 13100
 Wire Wire Line
-	23500 13100 23500 8200
+	23500 13100 23500 9750
 Wire Wire Line
-	3800 5750 3800 9900
+	3900 5750 3900 9900
 Wire Wire Line
-	12550 5350 24100 5350
+	12550 5350 24450 5350
 Wire Wire Line
-	13900 5400 24050 5400
+	13900 5400 24400 5400
 Wire Wire Line
-	14950 5450 24000 5450
+	14950 5450 24350 5450
 Wire Wire Line
-	16000 5550 23950 5550
+	16000 5500 24300 5500
 Wire Wire Line
-	18100 5650 23850 5650
+	18100 5600 24200 5600
 Wire Wire Line
-	17050 5600 23900 5600
+	17050 5550 24250 5550
 Wire Wire Line
-	19150 5700 23800 5700
+	19150 5650 24150 5650
 Wire Wire Line
-	3800 5750 11500 5750
+	3900 5750 11500 5750
 Wire Wire Line
 	3950 5800 10450 5800
@@
 	4250 9200 4250 12950
 Wire Wire Line
-	8400 9900 3800 9900
+	8400 9900 3900 9900
 Wire Wire Line
 	4200 6050 4200 10200
@@
 	8000 10200 4200 10200
 Wire Wire Line
-	23800 5700 23800 15400
-Wire Wire Line
-	23850 15450 8250 15450
+	24150 5650 24150 15400
 Wire Wire Line
-	23850 5650 23850 15450
+	24200 15450 8250 15450
 Wire Wire Line
-	23900 5600 23900 15500
+	24200 5600 24200 15450
 Wire Wire Line
-	23950 15550 8150 15550
+	24250 5550 24250 15500
 Wire Wire Line
-	23950 5550 23950 15550
+	24300 15550 8150 15550
 Wire Wire Line
-	24000 5450 24000 15650
+	24300 5500 24300 15550
 Wire Wire Line
-	24050 5400 24050 15700
+	24350 5450 24350 15650
 Wire Wire Line
-	24100 5350 24100 15750
+	24400 5400 24400 15700
 Wire Wire Line
-	8000 15750 24100 15750
+	24450 5350 24450 15750
 Wire Wire Line
-	8300 15400 23800 15400
+	8000 15750 24450 15750
 Wire Wire Line
-	8050 15700 24050 15700
+	8300 15400 24150 15400
 Wire Wire Line
-	8100 15650 24000 15650
+	8050 15700 24400 15700
 Wire Wire Line
-	8200 15500 23900 15500
+	8100 15650 24350 15650
 Wire Wire Line
-	23400 8150 23550 8150
+	8200 15500 24250 15500
 Wire Wire Line
-	23450 8200 23500 8200
-Wire Wire Line
-	23600 6800 23650 6800
-Wire Wire Line
-	23350 8100 23600 8100
-Wire Wire Line
-	23700 6750 23550 6750
-Wire Wire Line
-	23550 6750 23550 7300
-Wire Wire Line
-	23700 6750 23700 14900
+	23700 7300 23700 14900
 Text Notes 5100 6100 0    50   Italic 0
 Col_1\n
@@
 Text Notes 22300 5950 0    50   Italic 0
 Col-17
-Wire Wire Line
-	23250 7800 23250 8500
 Text Label 21100 6600 0    50   Italic 0
 LED_C1
@@
 	1    0    0    -1
 $EndComp
-Wire Wire Line
-	22300 5850 22300 6300
 Connection ~ 22300 7500
 Connection ~ 22300 6300
@@
 	1    0    0    -1
 $EndComp
-Wire Wire Line
-	20200 5850 20200 6300
 Connection ~ 20200 8750
 Connection ~ 20200 8150
@@
 	1    0    0    -1
 $EndComp
-Wire Wire Line
-	21250 5850 21250 6300
 Connection ~ 21250 8750
 Connection ~ 21250 8150
@@
 Connection ~ 20650 8500
 Wire Wire Line
-	23250 10700 23250 8500
-Wire Wire Line
-	14000 10700 23250 10700
-Wire Wire Line
-	23300 6600 23300 7200
+	14000 10700 22700 10700
 Wire Wire Line
 	18550 6600 19600 6600
@@
 Connection ~ 20650 9650
 Wire Wire Line
-	23200 9650 23200 10450
-Wire Wire Line
-	13950 10450 23200 10450
+	13950 10450 22600 10450
 Connection ~ 21400 6150
 Connection ~ 21400 7350
@@
 Connection ~ 21700 9050
 Wire Wire Line
-	21550 7900 23600 7900
-Wire Wire Line
 	21550 6700 23750 6700
 Wire Wire Line
-	21700 9050 23200 9050
+	21700 9050 22600 9050
 Wire Wire Line
-	21700 7800 23250 7800
+	21700 7800 22700 7800
 Wire Wire Line
-	21700 6600 23300 6600
+	21700 6600 22800 6600
 Connection ~ 19600 6600
 Wire Wire Line
@@
 Wire Wire Line
 	20650 6600 21700 6600
-Wire Wire Line
-	20500 9750 23450 9750
 $Comp
 L lee_mech_key_comp:SWITCH_PUSH PLUS
@@
 $EndComp
 Wire Wire Line
-	21550 9150 23400 9150
-Wire Wire Line
 	20500 9150 21550 9150
 Connection ~ 21550 9150
@@
 	22300 7500 22300 8750
 Wire Wire Line
-	20500 8550 23350 8550
-Wire Wire Line
 	22300 6300 22300 7500
 Wire Wire Line
-	20500 7300 23550 7300
+	20650 7200 22800 7200
+Wire Wire Line
+	20650 8500 22700 8500
+Wire Wire Line
+	20650 9650 22600 9650
+Wire Wire Line
+	11800 11000 11800 10450
+Connection ~ 13950 10450
+Wire Wire Line
+	14000 10700 13100 10700
+Wire Wire Line
+	11800 10450 13950 10450
+Wire Wire Line
+	13100 10700 13100 11250
+Wire Wire Line
+	22600 9050 22600 9650
+Connection ~ 22600 9650
+Wire Wire Line
+	22600 9650 22600 10450
+Wire Wire Line
+	22700 10700 22700 8500
+Connection ~ 22700 8500
+Wire Wire Line
+	22700 7800 22700 8500
+Wire Wire Line
+	22800 10850 22800 7200
+Wire Wire Line
+	22800 10850 16650 10850
+Connection ~ 22800 7200
+Wire Wire Line
+	22800 7200 22800 6600
+Wire Wire Line
+	21550 7900 23650 7900
+Wire Wire Line
+	20500 7300 23700 7300
+Wire Wire Line
+	20500 9750 23500 9750
+Wire Wire Line
+	21550 9150 23550 9150
+Wire Wire Line
+	20200 5700 24100 5700
+Wire Wire Line
+	24100 5700 24100 15350
+Wire Wire Line
+	24100 15350 8350 15350
+Wire Wire Line
+	20200 5700 20200 6300
+Wire Wire Line
+	20500 8550 23600 8550
+Wire Wire Line
+	8400 15300 24050 15300
+Wire Wire Line
+	24050 15300 24050 5750
+Wire Wire Line
+	24050 5750 21250 5750
+Wire Wire Line
+	21250 5750 21250 6300
+Wire Wire Line
+	22300 5800 24000 5800
 Wire Wire Line
-	20650 7200 23300 7200
+	24000 5800 24000 15250
 Wire Wire Line
-	20650 8500 23250 8500
+	24000 15250 8450 15250
 Wire Wire Line
-	20650 9650 23200 9650
+	22300 5800 22300 6300
 $EndSCHEMATC

Commit message: wiring completed
Parts:
- gave numbers to parts that had none: 30
- renumbered DEC to DEC1, DEL to DEL1, DEV to DEV1, END to END1, INS to INS1, MUL to MUL1, NUMLOCK to NUMLOCK1, PLUS to PLUS1, R_Enter to R_Enter1, R_minus to R_minus1
Connections:
- wire segments 829 -> 853
- no-connect marks 27 -> 24

Commit message: ab
Parts:
- FUNC1, MENU1: footprint sw_fprint_wLed:CHERRY_PCB_100H -> sw_fprint_wLed:CHERRY_PCB_125H
- MCU1: footprint sw_fprint_wLed:Teensy2.0++_footprint_assigned -> sw_fprint_wLed:Teensy2.0++_footprint_assigned_v2
- PLUS1, R_Enter1: footprint sw_fprint_wLed:CHERRY_PCB_100H -> sw_fprint_wLed:CHERRY_PCB_200V
Changed lines of the file:
@@
 EESchema Schematic File Version 4
 LIBS:power
+LIBS:device
 LIBS:74xx
+LIBS:audio
+LIBS:interface
 LIBS:main_board4-cache
 EELAYER 26 0
@@
 F 0 "MCU1" H 7600 14200 60  0000 C CNN
 F 1 "Teensy2.0++" H 7750 14100 60  0000 C CNN
-F 2 "sw_fprint_wLed:Teensy2.0++_footprint_assigned" H 7750 14250 60  0001 C CNN
+F 2 "sw_fprint_wLed:Teensy2.0++_footprint_assigned_v2" H 7750 14250 60  0001 C CNN
 F 3 "" H 7750 14250 60  0001 C CNN
 	1    7750 14250
@@
 F 0 "MENU1" H 14800 9460 50  0000 C CNN
 F 1 "SWITCH_PUSH" H 14650 9270 50  0001 C CNN
-F 2 "sw_fprint_wLed:CHERRY_PCB_100H" H 14650 9350 60  0001 C CNN
+F 2 "sw_fprint_wLed:CHERRY_PCB_125H" H 14650 9350 60  0001 C CNN
 F 3 "" H 14650 9350 60  0001 C CNN
 	1    14650 9350
@@
 F 0 "FUNC1" H 15850 9460 50  0000 C CNN
 F 1 "SWITCH_PUSH" H 15700 9270 50  0001 C CNN
-F 2 "sw_fprint_wLed:CHERRY_PCB_100H" H 15700 9350 60  0001 C CNN
+F 2 "sw_fprint_wLed:CHERRY_PCB_125H" H 15700 9350 60  0001 C CNN
 F 3 "" H 15700 9350 60  0001 C CNN
 	1    15700 9350
@@
 F 0 "R_Enter1" H 21100 9460 50  0000 C CNN
 F 1 "SWITCH_PUSH" H 20950 9270 50  0001 C CNN
-F 2 "sw_fprint_wLed:CHERRY_PCB_100H" H 20950 9350 60  0001 C CNN
+F 2 "sw_fprint_wLed:CHERRY_PCB_200V" H 20950 9350 60  0001 C CNN
 F 3 "" H 20950 9350 60  0001 C CNN
 	1    20950 9350
@@
 F 0 "PLUS1" H 22150 8860 50  0000 C CNN
 F 1 "SWITCH_PUSH" H 22000 8670 50  0001 C CNN
-F 2 "sw_fprint_wLed:CHERRY_PCB_100H" H 22000 8750 60  0001 C CNN
+F 2 "sw_fprint_wLed:CHERRY_PCB_200V" H 22000 8750 60  0001 C CNN
 F 3 "" H 22000 8750 60  0001 C CNN
 	1    22000 8750

Commit message: wring controller
Connections:
- net at MCU1.24 (B4): now also R_trans1.2; no longer R_trans3.2
- net at MCU1.26 (B6): now also R_trans3.2; no longer R_trans1.2
Changed lines of the file:
@@
 	6500 13750 6500 13250
 Wire Wire Line
-	7850 12900 7850 13350
-Wire Wire Line
 	7900 14450 7900 14750
 Wire Wire Line
@@
 	7100 11200 7100 12900
 Wire Wire Line
-	7100 12900 7850 12900
-Wire Wire Line
 	7100 11200 9550 11200
 Wire Wire Line
@@
 	7200 11700 7200 12800
 Wire Wire Line
-	7200 12800 7950 12800
-Wire Wire Line
-	7950 12800 7950 13350
+	7200 12800 7850 12800
 Wire Wire Line
 	7500 14650 7800 14650
@@
 Wire Wire Line
 	7850 14700 6500 14700
+Wire Wire Line
+	7950 12900 7950 13350
+Wire Wire Line
+	7100 12900 7950 12900
+Wire Wire Line
+	7850 13350 7850 12800
 $EndSCHEMATC
