File: main_board4.kicad_pcb (KiCad board)
At the start: 2 copper layers, 320 x 140 mm, 263 parts

Commit message: add new footprint
Parts:
- added DEC1: SWITCH_PUSH, sw_fprint_wLed:CHERRY_PCB_100H, F.Cu at (265.9, 216.7)
- added DEL1: SWITCH_PUSH, sw_fprint_wLed:CHERRY_PCB_100H, F.Cu at (301.3, 217.1)
- added DEV1: SWITCH_PUSH, sw_fprint_wLed:CHERRY_PCB_100H, F.Cu at (245.7, 217.1)
- added INS1: SWITCH_PUSH, sw_fprint_wLed:CHERRY_PCB_100H, F.Cu at (192.3, 212.1)
- added MENU1: SWITCH_PUSH, sw_fprint_wLed:CHERRY_PCB_100H, F.Cu at (171.1, 211.3)
- added MUL1: SWITCH_PUSH, sw_fprint_wLed:CHERRY_PCB_100H, F.Cu at (190.3, 235.5)
- added NO0: SWITCH_PUSH, sw_fprint_wLed:CHERRY_PCB_100H, F.Cu at (271.7, 238.3)
- added NO1: SWITCH_PUSH, sw_fprint_wLed:CHERRY_PCB_100H, F.Cu at (325.3, 219.1)
- added NO4: SWITCH_PUSH, sw_fprint_wLed:CHERRY_PCB_100H, F.Cu at (338.1, 241.8)
- added NO7: SWITCH_PUSH, sw_fprint_wLed:CHERRY_PCB_100H, F.Cu at (306.9, 262.5)
- added NUMLOCK1: SWITCH_PUSH, sw_fprint_wLed:CHERRY_PCB_100H, F.Cu at (205.2, 260.0)
- added No2: SWITCH_PUSH, sw_fprint_wLed:CHERRY_PCB_100H, F.Cu at (295.6, 241.1)
- added No3: SWITCH_PUSH, sw_fprint_wLed:CHERRY_PCB_100H, F.Cu at (315.1, 243.2)
- added No5: SWITCH_PUSH, sw_fprint_wLed:CHERRY_PCB_100H, F.Cu at (265.7, 262.0)
- added No6: SWITCH_PUSH, sw_fprint_wLed:CHERRY_PCB_100H, F.Cu at (288.1, 261.0)
- added No8: SWITCH_PUSH, sw_fprint_wLed:CHERRY_PCB_100H, F.Cu at (244.4, 259.7)
- added No9: SWITCH_PUSH, sw_fprint_wLed:CHERRY_PCB_100H, F.Cu at (225.1, 258.1)
- added PAUSE1: SWITCH_PUSH, sw_fprint_wLed:CHERRY_PCB_100H, F.Cu at (181.4, 262.6)
- added PLUS1: SWITCH_PUSH, sw_fprint_wLed:CHERRY_PCB_100H, F.Cu at (159.2, 260.2)
- added PRSCREEN1: SWITCH_PUSH, sw_fprint_wLed:CHERRY_PCB_100H, F.Cu at (165.7, 236.7)
- added R_Enter1: SWITCH_PUSH, sw_fprint_wLed:CHERRY_PCB_100H, F.Cu at (214.4, 233.7)
- added R_minus1: SWITCH_PUSH, sw_fprint_wLed:CHERRY_PCB_100H, F.Cu at (218.4, 207.1)
- renumbered DELETE1 to HOME1, RALT1 to MENU1, PAGEDOWN1 to NO4, PAGEUP1 to NO7, PRINTSCREEN1 to PAUSE1, INSERT1 to PRSCREEN1
Connections:
- net Net-(Aa1-Pad4) renamed /LED_C2
- BACKSPACE1 pad 4: Net-(BACKSPACE1-Pad4) -> /LED_C1
- Bb1 pad 4: Net-(Bb1-Pad4) -> /LED_C3
- COMMA1 pad 4: Net-(Bb1-Pad4) -> /LED_C3
- COMMAND1 pad 4: Net-(Bb1-Pad4) -> /LED_C3
- Cc1 pad 4: Net-(Bb1-Pad4) -> /LED_C3
- D1 pad 2: Net-(D1-Pad2) -> /Row_1
- D10 pad 2: Net-(D10-Pad2) -> /Row_4
- D11 pad 2: Net-(D11-Pad2) -> /Row_5
- D12 pad 2: Net-(D12-Pad2) -> /Row_6
- D13 pad 2: Net-(D1-Pad2) -> /Row_1
- D14 pad 2: Net-(D14-Pad2) -> /Row_2
- D15 pad 2: Net-(D15-Pad2) -> /Row_3
- D16 pad 2: Net-(D10-Pad2) -> /Row_4
- D17 pad 2: Net-(D11-Pad2) -> /Row_5
- D18 pad 2: Net-(D12-Pad2) -> /Row_6
- D19 pad 2: Net-(D1-Pad2) -> /Row_1
- D2 pad 2: Net-(D14-Pad2) -> /Row_2
- D20 pad 2: Net-(D14-Pad2) -> /Row_2
- D21 pad 2: Net-(D15-Pad2) -> /Row_3
- D22 pad 2: Net-(D10-Pad2) -> /Row_4
- D23 pad 2: Net-(D11-Pad2) -> /Row_5
- D24 pad 2: Net-(D12-Pad2) -> /Row_6
- D25 pad 2: Net-(D1-Pad2) -> /Row_1
- D26 pad 2: Net-(D14-Pad2) -> /Row_2
- D27 pad 2: Net-(D15-Pad2) -> /Row_3
- D28 pad 2: Net-(D10-Pad2) -> /Row_4
- D29 pad 2: Net-(D11-Pad2) -> /Row_5
- D3 pad 2: Net-(D15-Pad2) -> /Row_3
- D30 pad 2: Net-(D12-Pad2) -> /Row_6
- D31 pad 2: Net-(D1-Pad2) -> /Row_1
- D32 pad 2: Net-(D14-Pad2) -> /Row_2
- D33 pad 2: Net-(D15-Pad2) -> /Row_3
- D34 pad 2: Net-(D10-Pad2) -> /Row_4
- D35 pad 2: Net-(D11-Pad2) -> /Row_5
- D36 pad 2: Net-(D12-Pad2) -> /Row_6
- D37 pad 2: Net-(D1-Pad2) -> /Row_1
- D38 pad 2: Net-(D14-Pad2) -> /Row_2
- D39 pad 2: Net-(D15-Pad2) -> /Row_3
- D4 pad 2: Net-(D10-Pad2) -> /Row_4
- D40 pad 2: Net-(D10-Pad2) -> /Row_4
- D41 pad 2: Net-(D11-Pad2) -> /Row_5
- D42 pad 2: Net-(D12-Pad2) -> /Row_6
- D43 pad 2: Net-(D1-Pad2) -> /Row_1
- D44 pad 2: Net-(D14-Pad2) -> /Row_2
- D45 pad 2: Net-(D15-Pad2) -> /Row_3
- D46 pad 2: Net-(D10-Pad2) -> /Row_4
- D47 pad 2: Net-(D11-Pad2) -> /Row_5
- D48 pad 2: Net-(D12-Pad2) -> /Row_6
- D49 pad 2: Net-(D1-Pad2) -> /Row_1
- D5 pad 2: Net-(D11-Pad2) -> /Row_5
- D50 pad 2: Net-(D14-Pad2) -> /Row_2
- D51 pad 2: Net-(D15-Pad2) -> /Row_3
- D52 pad 2: Net-(D10-Pad2) -> /Row_4
- D53 pad 2: Net-(D11-Pad2) -> /Row_5
- D54 pad 2: Net-(D12-Pad2) -> /Row_6
- D55 pad 2: Net-(D1-Pad2) -> /Row_1
- D56 pad 2: Net-(D14-Pad2) -> /Row_2
- D57 pad 2: Net-(D15-Pad2) -> /Row_3
- D58 pad 2: Net-(D10-Pad2) -> /Row_4
- D59 pad 2: Net-(D11-Pad2) -> /Row_5
- D6 pad 2: Net-(D12-Pad2) -> /Row_6
- D60 pad 2: Net-(D12-Pad2) -> /Row_6
- D61 pad 2: Net-(D1-Pad2) -> /Row_1
- D62 pad 2: Net-(D14-Pad2) -> /Row_2
- D63 pad 2: Net-(D15-Pad2) -> /Row_3
- D64 pad 2: Net-(D10-Pad2) -> /Row_4
- D65 pad 2: Net-(D11-Pad2) -> /Row_5
- D66 pad 2: Net-(D12-Pad2) -> /Row_6
- D67 pad 2: Net-(D1-Pad2) -> /Row_1
- D68 pad 2: Net-(D14-Pad2) -> /Row_2
- D69 pad 2: Net-(D15-Pad2) -> /Row_3
- D7 pad 2: Net-(D1-Pad2) -> /Row_1
- D70 pad 2: Net-(D10-Pad2) -> /Row_4
- D71 pad 2: Net-(D11-Pad2) -> /Row_5
- D72 pad 2: Net-(D12-Pad2) -> /Row_6
- D73 pad 2: Net-(D1-Pad2) -> /Row_1
- D74 pad 2: Net-(D14-Pad2) -> /Row_2
- D75 pad 2: Net-(D15-Pad2) -> /Row_3
- D76 pad 2: Net-(D10-Pad2) -> /Row_4
- D77 pad 2: Net-(D11-Pad2) -> /Row_5
- D78 pad 2: Net-(D12-Pad2) -> /Row_6
- D79 pad 2: Net-(D1-Pad2) -> /Row_1
- D8 pad 2: Net-(D14-Pad2) -> /Row_2
- D80 pad 2: Net-(D14-Pad2) -> /Row_2
- D81 pad 2: Net-(D15-Pad2) -> /Row_3
- D82 pad 2: Net-(D10-Pad2) -> /Row_4
- D83 pad 2: Net-(D11-Pad2) -> /Row_5
- D84 pad 2: Net-(D12-Pad2) -> /Row_6
- D9 pad 2: Net-(D15-Pad2) -> /Row_3
- DOT1 pad 4: Net-(Bb1-Pad4) -> /LED_C3
- DOWN1 pad 1: Net-(D78-Pad1) -> Net-(D72-Pad1)
- DOWN1 pad 2: Net-(BACKSLASH1-Pad2) -> Net-(DOWN1-Pad2)
- DOWN1 pad 4: Net-(Bb1-Pad4) -> /LED_C3
- END1 pad 1: Net-(D83-Pad1) -> (no net)
- END1 pad 2: Net-(DELETE1-Pad2) -> Net-(DEC1-Pad2)
- END1 pad 3: Net-(END1-Pad3) -> (no net)
- END1 pad 4: Net-(Bb1-Pad4) -> /LED_C1
- EQUAL1 pad 4: Net-(BACKSPACE1-Pad4) -> /LED_C1
- ESC1 pad 4: Net-(BACKSPACE1-Pad4) -> /LED_C1
- F1 pad 4: Net-(BACKSPACE1-Pad4) -> /LED_C1
- F10 pad 4: Net-(BACKSPACE1-Pad4) -> /LED_C1
- F11 pad 4: Net-(BACKSPACE1-Pad4) -> /LED_C1
- F12 pad 4: Net-(BACKSPACE1-Pad4) -> /LED_C1
- F2 pad 4: Net-(BACKSPACE1-Pad4) -> /LED_C1
- F3 pad 4: Net-(BACKSPACE1-Pad4) -> /LED_C1
- F4 pad 4: Net-(BACKSPACE1-Pad4) -> /LED_C1
- F5 pad 4: Net-(BACKSPACE1-Pad4) -> /LED_C1
- F6 pad 4: Net-(BACKSPACE1-Pad4) -> /LED_C1
- F7 pad 4: Net-(BACKSPACE1-Pad4) -> /LED_C1
- F8 pad 4: Net-(BACKSPACE1-Pad4) -> /LED_C1
- F9 pad 4: Net-(BACKSPACE1-Pad4) -> /LED_C1
- FUNC1 pad 4: Net-(Bb1-Pad4) -> /LED_C3
- Ff1 pad 4: Net-(Bb1-Pad4) -> /LED_C3
- GRAVE1 pad 4: Net-(BACKSPACE1-Pad4) -> /LED_C1
- Gg1 pad 4: Net-(Bb1-Pad4) -> /LED_C3
- HOME1 pad 2: Net-(DELETE1-Pad2) -> Net-(HOME1-Pad2) (x2)
- HOME1 pad 3: Net-(DELETE1-Pad3) -> Net-(HOME1-Pad3)
- HOME1 pad 4: Net-(BACKSPACE1-Pad4) -> /LED_C1 (x2)
- HOME1 pad 1: Net-(D80-Pad1) -> Net-(D79-Pad1)
- Hh1 pad 4: Net-(Bb1-Pad4) -> /LED_C3
- Jj1 pad 4: Net-(Bb1-Pad4) -> /LED_C3
- LALT1 pad 4: Net-(Bb1-Pad4) -> /LED_C3
- LCTRL1 pad 4: Net-(Bb1-Pad4) -> /LED_C3
- LEFT1 pad 2: Net-(LEFT1-Pad2) -> Net-(DOWN1-Pad2)
- LEFT1 pad 4: Net-(Bb1-Pad4) -> /LED_C3
- LSHIFT1 pad 4: Net-(Bb1-Pad4) -> /LED_C3
- MCU1 pad 12: Net-(D1-Pad2) -> Net-(DEL1-Pad2)
- MCU1 pad 13: Net-(D14-Pad2) -> (no net)
- MCU1 pad 14: Net-(D15-Pad2) -> /Row_6
- MCU1 pad 2: Net-(F8-Pad2) -> Net-(COMMA1-Pad2)
- MCU1 pad 3: Net-(COMMA1-Pad2) -> Net-(DOT1-Pad2)
- MCU1 pad 39: Net-(MCU1-Pad39) -> Net-(F8-Pad2)
- MCU1 pad 4: Net-(DOT1-Pad2) -> Net-(EQUAL1-Pad2)
- MCU1 pad 40: Net-(D12-Pad2) -> (no net)
- MCU1 pad 41: Net-(D11-Pad2) -> (no net)
- MCU1 pad 42: Net-(D10-Pad2) -> /Row_1
- MCU1 pad 5: Net-(EQUAL1-Pad2) -> Net-(DOWN1-Pad2)
- MCU1 pad 6: Net-(LEFT1-Pad2) -> Net-(BACKSLASH1-Pad2)
- MCU1 pad 7: Net-(BACKSLASH1-Pad2) -> Net-(HOME1-Pad2)
- MCU1 pad 8: Net-(DELETE1-Pad2) -> (no net)
- MENU1 pad 4: Net-(Bb1-Pad4) -> /LED_C3
- MINUS1 pad 4: Net-(BACKSPACE1-Pad4) -> /LED_C1
- Mm1 pad 4: Net-(Bb1-Pad4) -> /LED_C3
- NO4 pad 2: Net-(DELETE1-Pad2) -> Net-(HOME1-Pad2)
- NO7 pad 2: Net-(DELETE1-Pad2) -> Net-(HOME1-Pad2)
- Nn1 pad 4: Net-(Bb1-Pad4) -> /LED_C3
- ONE1 pad 4: Net-(BACKSPACE1-Pad4) -> /LED_C1
- PAUSE1 pad 2: Net-(LEFT1-Pad2) -> Net-(DOWN1-Pad2)
- PAUSE1 pad 4: Net-(BACKSPACE1-Pad4) -> /LED_C1
- PRSCREEN1 pad 4: Net-(BACKSPACE1-Pad4) -> /LED_C1
- P_jump_trans1 pad 1: Net-(Bb1-Pad4) -> /LED_C3
- P_jump_trans3 pad 1: Net-(BACKSPACE1-Pad4) -> /LED_C1
- QUOTE1 pad 2: Net-(LEFT1-Pad2) -> Net-(DOWN1-Pad2)
- R72 pad 2: Net-(R72-Pad2) -> Net-(DOWN1-Pad3)
- R78 pad 2: Net-(DOWN1-Pad3) -> Net-(R78-Pad2)
- R79 pad 2: Net-(DELETE1-Pad3) -> Net-(HOME1-Pad3)
- R80 pad 2: Net-(HOME1-Pad3) -> Net-(NUMLOCK1-Pad3)
- R83 pad 2: Net-(END1-Pad3) -> Net-(NO1-Pad3)
- R84 pad 2: Net-(R84-Pad2) -> Net-(NO0-Pad3)
- RBRAKET1 pad 2: Net-(LEFT1-Pad2) -> Net-(DOWN1-Pad2)
- RBRAKET1 pad 4: Net-(BACKSPACE1-Pad4) -> /LED_C1
- RCTRL1 pad 2: Net-(LEFT1-Pad2) -> (no net)
- RCTRL1 pad 3: Net-(R72-Pad2) -> (no net)
- RCTRL1 pad 4: Net-(Bb1-Pad4) -> (no net)
- RIGHT1 pad 1: Net-(D84-Pad1) -> Net-(D78-Pad1)
- RIGHT1 pad 2: Net-(DELETE1-Pad2) -> Net-(BACKSLASH1-Pad2)
- RIGHT1 pad 3: Net-(R84-Pad2) -> Net-(R78-Pad2)
- RIGHT1 pad 4: Net-(Bb1-Pad4) -> /LED_C3
- RSHIFT1 pad 2: Net-(LEFT1-Pad2) -> Net-(DOWN1-Pad2)
- SEVEN7 pad 4: Net-(BACKSPACE1-Pad4) -> /LED_C1
- SIX6 pad 4: Net-(BACKSPACE1-Pad4) -> /LED_C1
- SLASH1 pad 4: Net-(Bb1-Pad4) -> /LED_C3
- SPACE1 pad 4: Net-(Bb1-Pad4) -> /LED_C3
- THREE3 pad 4: Net-(BACKSPACE1-Pad4) -> /LED_C1
- TWO2 pad 4: Net-(BACKSPACE1-Pad4) -> /LED_C1
- Transistor1 pad 2: Net-(Bb1-Pad4) -> /LED_C3
- Transistor3 pad 2: Net-(BACKSPACE1-Pad4) -> /LED_C1
- UP1 pad 4: Net-(Bb1-Pad4) -> /LED_C3
- Vv1 pad 4: Net-(Bb1-Pad4) -> /LED_C3
- Xx1 pad 4: Net-(Bb1-Pad4) -> /LED_C3
- Yy1 pad 4: Net-(Bb1-Pad4) -> /LED_C3
- ZERO0 pad 4: Net-(BACKSPACE1-Pad4) -> /LED_C1
- Zz1 pad 4: Net-(Bb1-Pad4) -> /LED_C3
- ext_1 pad 7: Net-(MCU1-Pad39) -> (no net)
Routing:
- net Net-(BACKSPACE1-Pad4): track 1182.1 -> 0.00 mm
- net Net-(Bb1-Pad4): track 1150.2 -> 0.00 mm
- net /LED_C2: track 825.7 -> 0.00 mm
- net Net-(D15-Pad2): track 481.0 -> 0.00 mm
- net Net-(D14-Pad2): track 475.8 -> 0.00 mm
- net Net-(D12-Pad2): track 394.4 -> 0.00 mm
- net Net-(D1-Pad2): track 387.1 -> 0.00 mm
- net Net-(D11-Pad2): track 384.5 -> 0.00 mm
- net Net-(D10-Pad2): track 372.2 -> 0.00 mm
- net Net-(Bb1-Pad2): track 211.9 -> 0.00 mm
- net Net-(F6-Pad2): track 186.2 -> 0.00 mm
- net Net-(Cc1-Pad2): track 177.3 -> 0.00 mm
- net Net-(F4-Pad2): track 156.1 -> 0.00 mm
- net Net-(CAPLOCK1-Pad2): track 144.9 -> 0.00 mm
- net Net-(LEFT1-Pad2): track 139.1 -> 0.00 mm
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- removed copper zone on B.Cu, net Net-(MCU1-Pad46)
- removed copper zone on F.Cu, net Net-(MCU1-Pad49)

Commit message: keep old pcb design
Parts:
- removed DEC1, DEL1, DEV1, INS1, MENU1, MUL1, NO0, NO1, NO4, NO7, NUMLOCK1, No2, No3, No5, No6, No8, No9, PAUSE1, PLUS1, PRSCREEN1, R_Enter1, R_minus1: SWITCH_PUSH, sw_fprint_wLed:CHERRY_PCB_100H
- renumbered HOME1 to DELETE1, PRSCREEN1 to INSERT1, NO4 to PAGEDOWN1, NO7 to PAGEUP1, PAUSE1 to PRINTSCREEN1, MENU1 to RALT1
Connections:
- net /LED_C2 renamed Net-(Aa1-Pad4)
- BACKSPACE1 pad 4: /LED_C1 -> Net-(BACKSPACE1-Pad4)
- Bb1 pad 4: /LED_C3 -> Net-(Bb1-Pad4)
- COMMA1 pad 4: /LED_C3 -> Net-(Bb1-Pad4)
- COMMAND1 pad 4: /LED_C3 -> Net-(Bb1-Pad4)
- Cc1 pad 4: /LED_C3 -> Net-(Bb1-Pad4)
- D1 pad 2: /Row_1 -> Net-(D1-Pad2)
- D10 pad 2: /Row_4 -> Net-(D10-Pad2)
- D11 pad 2: /Row_5 -> Net-(D11-Pad2)
- D12 pad 2: /Row_6 -> Net-(D12-Pad2)
- D13 pad 2: /Row_1 -> Net-(D1-Pad2)
- D14 pad 2: /Row_2 -> Net-(D14-Pad2)
- D15 pad 2: /Row_3 -> Net-(D15-Pad2)
- D16 pad 2: /Row_4 -> Net-(D10-Pad2)
- D17 pad 2: /Row_5 -> Net-(D11-Pad2)
- D18 pad 2: /Row_6 -> Net-(D12-Pad2)
- D19 pad 2: /Row_1 -> Net-(D1-Pad2)
- D2 pad 2: /Row_2 -> Net-(D14-Pad2)
- D20 pad 2: /Row_2 -> Net-(D14-Pad2)
- D21 pad 2: /Row_3 -> Net-(D15-Pad2)
- D22 pad 2: /Row_4 -> Net-(D10-Pad2)
- D23 pad 2: /Row_5 -> Net-(D11-Pad2)
- D24 pad 2: /Row_6 -> Net-(D12-Pad2)
- D25 pad 2: /Row_1 -> Net-(D1-Pad2)
- D26 pad 2: /Row_2 -> Net-(D14-Pad2)
- D27 pad 2: /Row_3 -> Net-(D15-Pad2)
- D28 pad 2: /Row_4 -> Net-(D10-Pad2)
- D29 pad 2: /Row_5 -> Net-(D11-Pad2)
- D3 pad 2: /Row_3 -> Net-(D15-Pad2)
- D30 pad 2: /Row_6 -> Net-(D12-Pad2)
- D31 pad 2: /Row_1 -> Net-(D1-Pad2)
- D32 pad 2: /Row_2 -> Net-(D14-Pad2)
- D33 pad 2: /Row_3 -> Net-(D15-Pad2)
- D34 pad 2: /Row_4 -> Net-(D10-Pad2)
- D35 pad 2: /Row_5 -> Net-(D11-Pad2)
- D36 pad 2: /Row_6 -> Net-(D12-Pad2)
- D37 pad 2: /Row_1 -> Net-(D1-Pad2)
- D38 pad 2: /Row_2 -> Net-(D14-Pad2)
- D39 pad 2: /Row_3 -> Net-(D15-Pad2)
- D4 pad 2: /Row_4 -> Net-(D10-Pad2)
- D40 pad 2: /Row_4 -> Net-(D10-Pad2)
- D41 pad 2: /Row_5 -> Net-(D11-Pad2)
- D42 pad 2: /Row_6 -> Net-(D12-Pad2)
- D43 pad 2: /Row_1 -> Net-(D1-Pad2)
- D44 pad 2: /Row_2 -> Net-(D14-Pad2)
- D45 pad 2: /Row_3 -> Net-(D15-Pad2)
- D46 pad 2: /Row_4 -> Net-(D10-Pad2)
- D47 pad 2: /Row_5 -> Net-(D11-Pad2)
- D48 pad 2: /Row_6 -> Net-(D12-Pad2)
- D49 pad 2: /Row_1 -> Net-(D1-Pad2)
- D5 pad 2: /Row_5 -> Net-(D11-Pad2)
- D50 pad 2: /Row_2 -> Net-(D14-Pad2)
- D51 pad 2: /Row_3 -> Net-(D15-Pad2)
- D52 pad 2: /Row_4 -> Net-(D10-Pad2)
- D53 pad 2: /Row_5 -> Net-(D11-Pad2)
- D54 pad 2: /Row_6 -> Net-(D12-Pad2)
- D55 pad 2: /Row_1 -> Net-(D1-Pad2)
- D56 pad 2: /Row_2 -> Net-(D14-Pad2)
- D57 pad 2: /Row_3 -> Net-(D15-Pad2)
- D58 pad 2: /Row_4 -> Net-(D10-Pad2)
- D59 pad 2: /Row_5 -> Net-(D11-Pad2)
- D6 pad 2: /Row_6 -> Net-(D12-Pad2)
- D60 pad 2: /Row_6 -> Net-(D12-Pad2)
- D61 pad 2: /Row_1 -> Net-(D1-Pad2)
- D62 pad 2: /Row_2 -> Net-(D14-Pad2)
- D63 pad 2: /Row_3 -> Net-(D15-Pad2)
- D64 pad 2: /Row_4 -> Net-(D10-Pad2)
- D65 pad 2: /Row_5 -> Net-(D11-Pad2)
- D66 pad 2: /Row_6 -> Net-(D12-Pad2)
- D67 pad 2: /Row_1 -> Net-(D1-Pad2)
- D68 pad 2: /Row_2 -> Net-(D14-Pad2)
- D69 pad 2: /Row_3 -> Net-(D15-Pad2)
- D7 pad 2: /Row_1 -> Net-(D1-Pad2)
- D70 pad 2: /Row_4 -> Net-(D10-Pad2)
- D71 pad 2: /Row_5 -> Net-(D11-Pad2)
- D72 pad 2: /Row_6 -> Net-(D12-Pad2)
- D73 pad 2: /Row_1 -> Net-(D1-Pad2)
- D74 pad 2: /Row_2 -> Net-(D14-Pad2)
- D75 pad 2: /Row_3 -> Net-(D15-Pad2)
- D76 pad 2: /Row_4 -> Net-(D10-Pad2)
- D77 pad 2: /Row_5 -> Net-(D11-Pad2)
- D78 pad 2: /Row_6 -> Net-(D12-Pad2)
- D79 pad 2: /Row_1 -> Net-(D1-Pad2)
- D8 pad 2: /Row_2 -> Net-(D14-Pad2)
- D80 pad 2: /Row_2 -> Net-(D14-Pad2)
- D81 pad 2: /Row_3 -> Net-(D15-Pad2)
- D82 pad 2: /Row_4 -> Net-(D10-Pad2)
- D83 pad 2: /Row_5 -> Net-(D11-Pad2)
- D84 pad 2: /Row_6 -> Net-(D12-Pad2)
- D9 pad 2: /Row_3 -> Net-(D15-Pad2)
- DELETE1 pad 2: Net-(HOME1-Pad2) -> Net-(DELETE1-Pad2)
- DELETE1 pad 3: Net-(HOME1-Pad3) -> Net-(DELETE1-Pad3)
- DELETE1 pad 4: /LED_C1 -> Net-(BACKSPACE1-Pad4)
- DOT1 pad 4: /LED_C3 -> Net-(Bb1-Pad4)
- DOWN1 pad 1: Net-(D72-Pad1) -> Net-(D78-Pad1)
- DOWN1 pad 2: Net-(DOWN1-Pad2) -> Net-(BACKSLASH1-Pad2)
- DOWN1 pad 4: /LED_C3 -> Net-(Bb1-Pad4)
- END1 pad 1: (no net) -> Net-(D83-Pad1)
- END1 pad 2: Net-(DEC1-Pad2) -> Net-(DELETE1-Pad2)
- END1 pad 3: (no net) -> Net-(END1-Pad3)
- END1 pad 4: /LED_C1 -> Net-(Bb1-Pad4)
- EQUAL1 pad 4: /LED_C1 -> Net-(BACKSPACE1-Pad4)
- ESC1 pad 4: /LED_C1 -> Net-(BACKSPACE1-Pad4)
- F1 pad 4: /LED_C1 -> Net-(BACKSPACE1-Pad4)
- F10 pad 4: /LED_C1 -> Net-(BACKSPACE1-Pad4)
- F11 pad 4: /LED_C1 -> Net-(BACKSPACE1-Pad4)
- F12 pad 4: /LED_C1 -> Net-(BACKSPACE1-Pad4)
- F2 pad 4: /LED_C1 -> Net-(BACKSPACE1-Pad4)
- F3 pad 4: /LED_C1 -> Net-(BACKSPACE1-Pad4)
- F4 pad 4: /LED_C1 -> Net-(BACKSPACE1-Pad4)
- F5 pad 4: /LED_C1 -> Net-(BACKSPACE1-Pad4)
- F6 pad 4: /LED_C1 -> Net-(BACKSPACE1-Pad4)
- F7 pad 4: /LED_C1 -> Net-(BACKSPACE1-Pad4)
- F8 pad 4: /LED_C1 -> Net-(BACKSPACE1-Pad4)
- F9 pad 4: /LED_C1 -> Net-(BACKSPACE1-Pad4)
- FUNC1 pad 4: /LED_C3 -> Net-(Bb1-Pad4)
- Ff1 pad 4: /LED_C3 -> Net-(Bb1-Pad4)
- GRAVE1 pad 4: /LED_C1 -> Net-(BACKSPACE1-Pad4)
- Gg1 pad 4: /LED_C3 -> Net-(Bb1-Pad4)
- HOME1 pad 1: Net-(D79-Pad1) -> Net-(D80-Pad1)
- HOME1 pad 2: Net-(HOME1-Pad2) -> Net-(DELETE1-Pad2)
- HOME1 pad 4: /LED_C1 -> Net-(BACKSPACE1-Pad4)
- Hh1 pad 4: /LED_C3 -> Net-(Bb1-Pad4)
- INSERT1 pad 4: /LED_C1 -> Net-(BACKSPACE1-Pad4)
- Jj1 pad 4: /LED_C3 -> Net-(Bb1-Pad4)
- LALT1 pad 4: /LED_C3 -> Net-(Bb1-Pad4)
- LCTRL1 pad 4: /LED_C3 -> Net-(Bb1-Pad4)
- LEFT1 pad 2: Net-(DOWN1-Pad2) -> Net-(LEFT1-Pad2)
- LEFT1 pad 4: /LED_C3 -> Net-(Bb1-Pad4)
- LSHIFT1 pad 4: /LED_C3 -> Net-(Bb1-Pad4)
- MCU1 pad 12: Net-(DEL1-Pad2) -> Net-(D1-Pad2)
- MCU1 pad 13: (no net) -> Net-(D14-Pad2)
- MCU1 pad 14: /Row_6 -> Net-(D15-Pad2)
- MCU1 pad 2: Net-(COMMA1-Pad2) -> Net-(F8-Pad2)
- MCU1 pad 3: Net-(DOT1-Pad2) -> Net-(COMMA1-Pad2)
- MCU1 pad 39: Net-(F8-Pad2) -> Net-(MCU1-Pad39)
- MCU1 pad 4: Net-(EQUAL1-Pad2) -> Net-(DOT1-Pad2)
- MCU1 pad 40: (no net) -> Net-(D12-Pad2)
- MCU1 pad 41: (no net) -> Net-(D11-Pad2)
- MCU1 pad 42: /Row_1 -> Net-(D10-Pad2)
- MCU1 pad 5: Net-(DOWN1-Pad2) -> Net-(EQUAL1-Pad2)
- MCU1 pad 6: Net-(BACKSLASH1-Pad2) -> Net-(LEFT1-Pad2)
- MCU1 pad 7: Net-(HOME1-Pad2) -> Net-(BACKSLASH1-Pad2)
- MCU1 pad 8: (no net) -> Net-(DELETE1-Pad2)
- MINUS1 pad 4: /LED_C1 -> Net-(BACKSPACE1-Pad4)
- Mm1 pad 4: /LED_C3 -> Net-(Bb1-Pad4)
- Nn1 pad 4: /LED_C3 -> Net-(Bb1-Pad4)
- ONE1 pad 4: /LED_C1 -> Net-(BACKSPACE1-Pad4)
- PAGEDOWN1 pad 2: Net-(HOME1-Pad2) -> Net-(DELETE1-Pad2)
- PAGEUP1 pad 2: Net-(HOME1-Pad2) -> Net-(DELETE1-Pad2)
- PRINTSCREEN1 pad 2: Net-(DOWN1-Pad2) -> Net-(LEFT1-Pad2)
- PRINTSCREEN1 pad 4: /LED_C1 -> Net-(BACKSPACE1-Pad4)
- P_jump_trans1 pad 1: /LED_C3 -> Net-(Bb1-Pad4)
- P_jump_trans3 pad 1: /LED_C1 -> Net-(BACKSPACE1-Pad4)
- QUOTE1 pad 2: Net-(DOWN1-Pad2) -> Net-(LEFT1-Pad2)
- R72 pad 2: Net-(DOWN1-Pad3) -> Net-(R72-Pad2)
- R78 pad 2: Net-(R78-Pad2) -> Net-(DOWN1-Pad3)
- R79 pad 2: Net-(HOME1-Pad3) -> Net-(DELETE1-Pad3)
- R80 pad 2: Net-(NUMLOCK1-Pad3) -> Net-(HOME1-Pad3)
- R83 pad 2: Net-(NO1-Pad3) -> Net-(END1-Pad3)
- R84 pad 2: Net-(NO0-Pad3) -> Net-(R84-Pad2)
- RALT1 pad 4: /LED_C3 -> Net-(Bb1-Pad4)
- RBRAKET1 pad 2: Net-(DOWN1-Pad2) -> Net-(LEFT1-Pad2)
- RBRAKET1 pad 4: /LED_C1 -> Net-(BACKSPACE1-Pad4)
- RCTRL1 pad 2: (no net) -> Net-(LEFT1-Pad2)
- RCTRL1 pad 3: (no net) -> Net-(R72-Pad2)
- RCTRL1 pad 4: (no net) -> Net-(Bb1-Pad4)
- RIGHT1 pad 1: Net-(D78-Pad1) -> Net-(D84-Pad1)
- RIGHT1 pad 2: Net-(BACKSLASH1-Pad2) -> Net-(DELETE1-Pad2)
- RIGHT1 pad 3: Net-(R78-Pad2) -> Net-(R84-Pad2)
- RIGHT1 pad 4: /LED_C3 -> Net-(Bb1-Pad4)
- RSHIFT1 pad 2: Net-(DOWN1-Pad2) -> Net-(LEFT1-Pad2)
- SEVEN7 pad 4: /LED_C1 -> Net-(BACKSPACE1-Pad4)
- SIX6 pad 4: /LED_C1 -> Net-(BACKSPACE1-Pad4)
- SLASH1 pad 4: /LED_C3 -> Net-(Bb1-Pad4)
- SPACE1 pad 4: /LED_C3 -> Net-(Bb1-Pad4)
- THREE3 pad 4: /LED_C1 -> Net-(BACKSPACE1-Pad4)
- TWO2 pad 4: /LED_C1 -> Net-(BACKSPACE1-Pad4)
- Transistor1 pad 2: /LED_C3 -> Net-(Bb1-Pad4)
- Transistor3 pad 2: /LED_C1 -> Net-(BACKSPACE1-Pad4)
- UP1 pad 4: /LED_C3 -> Net-(Bb1-Pad4)
- Vv1 pad 4: /LED_C3 -> Net-(Bb1-Pad4)
- Xx1 pad 4: /LED_C3 -> Net-(Bb1-Pad4)
- Yy1 pad 4: /LED_C3 -> Net-(Bb1-Pad4)
- ZERO0 pad 4: /LED_C1 -> Net-(BACKSPACE1-Pad4)
- Zz1 pad 4: /LED_C3 -> Net-(Bb1-Pad4)
- ext_1 pad 7: (no net) -> Net-(MCU1-Pad39)
Routing:
- net Net-(BACKSPACE1-Pad4): track 0.00 -> 1182.1 mm
- net Net-(Bb1-Pad4): track 0.00 -> 1150.2 mm
- net Net-(Aa1-Pad4): track 0.00 -> 825.7 mm
- net Net-(D15-Pad2): track 0.00 -> 481.0 mm
- net Net-(D14-Pad2): track 0.00 -> 475.8 mm
- net Net-(D12-Pad2): track 0.00 -> 394.4 mm
- net Net-(D1-Pad2): track 0.00 -> 387.1 mm
- net Net-(D11-Pad2): track 0.00 -> 384.5 mm
- net Net-(D10-Pad2): track 0.00 -> 372.2 mm
- net Net-(Bb1-Pad2): track 0.00 -> 211.9 mm
- net Net-(F6-Pad2): track 0.00 -> 186.2 mm
- net Net-(Cc1-Pad2): track 0.00 -> 177.3 mm
- net Net-(F4-Pad2): track 0.00 -> 156.1 mm
- net Net-(CAPLOCK1-Pad2): track 0.00 -> 144.9 mm
- net Net-(LEFT1-Pad2): track 0.00 -> 139.1 mm
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- added copper zone on B.Cu, net Net-(MCU1-Pad46)
- added copper zone on F.Cu, net Net-(MCU1-Pad49)

Commit message: ab
Parts:
- removed DELETE1, INSERT1, PAGEDOWN1, PAGEUP1, PRINTSCREEN1, RALT1, RCTRL1: SWITCH_PUSH, sw_fprint_wLed:CHERRY_PCB_100H
- added D85: DIODE, Diode_SMD:D_MiniMELF, F.Cu at (177.0, 227.8)
- added D86: DIODE, Diode_SMD:D_MiniMELF, F.Cu at (177.0, 230.1)
- added D87: DIODE, Diode_SMD:D_MiniMELF, F.Cu at (182.3, 227.8)
- added D88: DIODE, Diode_SMD:D_MiniMELF, F.Cu at (177.0, 232.3)
- added D89: DIODE, Diode_SMD:D_MiniMELF, F.Cu at (182.3, 230.1)
- added D90: DIODE, Diode_SMD:D_MiniMELF, F.Cu at (177.0, 234.6)
- added D91: DIODE, Diode_SMD:D_MiniMELF, F.Cu at (187.7, 227.8)
- added D92: DIODE, Diode_SMD:D_MiniMELF, F.Cu at (177.0, 236.8)
- added D93: DIODE, Diode_SMD:D_MiniMELF, F.Cu at (182.3, 232.3)
- added D94: DIODE, Diode_SMD:D_MiniMELF, F.Cu at (187.7, 230.1)
- added D95: DIODE, Diode_SMD:D_MiniMELF, F.Cu at (182.3, 234.6)
- added D96: DIODE, Diode_SMD:D_MiniMELF, F.Cu at (177.0, 239.1)
- added D97: DIODE, Diode_SMD:D_MiniMELF, F.Cu at (193.0, 227.8)
- added D98: DIODE, Diode_SMD:D_MiniMELF, F.Cu at (182.3, 236.8)
- added D99: DIODE, Diode_SMD:D_MiniMELF, F.Cu at (187.7, 232.3)
- added DEC1: SWITCH_PUSH, sw_fprint_wLed:CHERRY_PCB_100H, F.Cu at (426.7, 177.2)
- added DEL1: SWITCH_PUSH, sw_fprint_wLed:CHERRY_PCB_100H, F.Cu at (448.1, 70.1)
- added DEV1: SWITCH_PUSH, sw_fprint_wLed:CHERRY_PCB_100H, F.Cu at (424.3, 110.6)
- added INS1: SWITCH_PUSH, sw_fprint_wLed:CHERRY_PCB_100H, F.Cu at (479.1, 79.6)
- added MENU1: SWITCH_PUSH, sw_fprint_wLed:CHERRY_PCB_125H, F.Cu at (267.2, 172.5)
- added MUL1: SWITCH_PUSH, sw_fprint_wLed:CHERRY_PCB_100H, F.Cu at (441.0, 89.1)
- added NO0: SWITCH_PUSH, sw_fprint_wLed:CHERRY_PCB_100H, F.Cu at (474.3, 193.9)
- added NO1: SWITCH_PUSH, sw_fprint_wLed:CHERRY_PCB_100H, F.Cu at (405.3, 227.2)
- added NO4: SWITCH_PUSH, sw_fprint_wLed:CHERRY_PCB_100H, F.Cu at (474.3, 227.2)
- added NO7, NUMLOCK1, No5, No6, No8, No9, PAUSE1, PRSCREEN1: SWITCH_PUSH, sw_fprint_wLed:CHERRY_PCB_100H, F.Cu at (485.0, 152.6)
- added No2: SWITCH_PUSH, sw_fprint_wLed:CHERRY_PCB_100H, F.Cu at (429.1, 220.1)
- added No3: SWITCH_PUSH, sw_fprint_wLed:CHERRY_PCB_100H, F.Cu at (455.3, 220.1)
- added PLUS1: SWITCH_PUSH, sw_fprint_wLed:CHERRY_PCB_200V, F.Cu at (448.1, 120.1)
- added R85: R, Resistor_SMD:R_0805_2012Metric, F.Cu at (192.1, 229.9)
- added R86: R, Resistor_SMD:R_0805_2012Metric, F.Cu at (186.7, 234.4)
- added R87: R, Resistor_SMD:R_0805_2012Metric, F.Cu at (181.4, 238.9)
- added R88: R, Resistor_SMD:R_0805_2012Metric, F.Cu at (184.8, 238.9)
- added R89: R, Resistor_SMD:R_0805_2012Metric, F.Cu at (190.1, 234.4)
- added R90: R, Resistor_SMD:R_0805_2012Metric, F.Cu at (186.7, 236.4)
- added R91: R, Resistor_SMD:R_0805_2012Metric, F.Cu at (192.1, 231.9)
- added R92: R, Resistor_SMD:R_0805_2012Metric, F.Cu at (195.5, 229.9)
- added R93: R, Resistor_SMD:R_0805_2012Metric, F.Cu at (188.2, 238.3)
- added R94: R, Resistor_SMD:R_0805_2012Metric, F.Cu at (190.1, 236.4)
- added R95: R, Resistor_SMD:R_0805_2012Metric, F.Cu at (193.5, 233.8)
- added R96: R, Resistor_SMD:R_0805_2012Metric, F.Cu at (195.5, 231.9)
- added R97: R, Resistor_SMD:R_0805_2012Metric, F.Cu at (191.6, 238.3)
- added R98: R, Resistor_SMD:R_0805_2012Metric, F.Cu at (193.5, 235.8)
- added R99: R, Resistor_SMD:R_0805_2012Metric, F.Cu at (196.9, 233.8)
- added R_Enter1: SWITCH_PUSH, sw_fprint_wLed:CHERRY_PCB_200V, F.Cu at (448.1, 158.2)
- added R_minus1: SWITCH_PUSH, sw_fprint_wLed:CHERRY_PCB_100H, F.Cu at (421.9, 93.9)
- FUNC1: footprint sw_fprint_wLed:CHERRY_PCB_100H -> sw_fprint_wLed:CHERRY_PCB_125H
- MCU1: footprint sw_fprint_wLed:Teensy2.0++_footprint_assigned -> sw_fprint_wLed:Teensy2.0++_footprint_assigned_v2
- SPACE1: footprint sw_fprint_wLed:CHERRY_PCB_625H -> sw_fprint_wLed:CHERRY_PCB_650H
- moved END1 101.5 mm to (419.6, 74.8), turned to 0 degrees
- moved HOME1 47.9 mm to (398.1, 74.8), turned to 0 degrees
- moved FUNC1 11.9 mm to (291.0, 172.5)
- moved SPACE1 2.38 mm to (193.3, 172.5)
Connections:
- net Net-(Aa1-Pad4) renamed /LED_C2
- BACKSPACE1 pad 4: Net-(BACKSPACE1-Pad4) -> /LED_C1
- Bb1 pad 4: Net-(Bb1-Pad4) -> /LED_C3
- COMMA1 pad 4: Net-(Bb1-Pad4) -> /LED_C3
- COMMAND1 pad 4: Net-(Bb1-Pad4) -> /LED_C3
- Cc1 pad 4: Net-(Bb1-Pad4) -> /LED_C3
- D1 pad 2: Net-(D1-Pad2) -> /Row_1
- D10 pad 2: Net-(D10-Pad2) -> /Row_4
- D11 pad 2: Net-(D11-Pad2) -> /Row_5
- D12 pad 2: Net-(D12-Pad2) -> /Row_6
- D13 pad 2: Net-(D1-Pad2) -> /Row_1
- D14 pad 2: Net-(D14-Pad2) -> /Row_2
- D15 pad 2: Net-(D15-Pad2) -> /Row_3
- D16 pad 2: Net-(D10-Pad2) -> /Row_4
- D17 pad 2: Net-(D11-Pad2) -> /Row_5
- D18 pad 2: Net-(D12-Pad2) -> /Row_6
- D19 pad 2: Net-(D1-Pad2) -> /Row_1
- D2 pad 2: Net-(D14-Pad2) -> /Row_2
- D20 pad 2: Net-(D14-Pad2) -> /Row_2
- D21 pad 2: Net-(D15-Pad2) -> /Row_3
- D22 pad 2: Net-(D10-Pad2) -> /Row_4
- D23 pad 2: Net-(D11-Pad2) -> /Row_5
- D24 pad 2: Net-(D12-Pad2) -> /Row_6
- D25 pad 2: Net-(D1-Pad2) -> /Row_1
- D26 pad 2: Net-(D14-Pad2) -> /Row_2
- D27 pad 2: Net-(D15-Pad2) -> /Row_3
- D28 pad 2: Net-(D10-Pad2) -> /Row_4
- D29 pad 2: Net-(D11-Pad2) -> /Row_5
- D3 pad 2: Net-(D15-Pad2) -> /Row_3
- D30 pad 2: Net-(D12-Pad2) -> /Row_6
- D31 pad 2: Net-(D1-Pad2) -> /Row_1
- D32 pad 2: Net-(D14-Pad2) -> /Row_2
- D33 pad 2: Net-(D15-Pad2) -> /Row_3
- D34 pad 2: Net-(D10-Pad2) -> /Row_4
- D35 pad 2: Net-(D11-Pad2) -> /Row_5
- D36 pad 2: Net-(D12-Pad2) -> /Row_6
- D37 pad 2: Net-(D1-Pad2) -> /Row_1
- D38 pad 2: Net-(D14-Pad2) -> /Row_2
- D39 pad 2: Net-(D15-Pad2) -> /Row_3
- D4 pad 2: Net-(D10-Pad2) -> /Row_4
- D40 pad 2: Net-(D10-Pad2) -> /Row_4
- D41 pad 2: Net-(D11-Pad2) -> /Row_5
- D42 pad 2: Net-(D12-Pad2) -> /Row_6
- D43 pad 2: Net-(D1-Pad2) -> /Row_1
- D44 pad 2: Net-(D14-Pad2) -> /Row_2
- D45 pad 2: Net-(D15-Pad2) -> /Row_3
- D46 pad 2: Net-(D10-Pad2) -> /Row_4
- D47 pad 2: Net-(D11-Pad2) -> /Row_5
- D48 pad 2: Net-(D12-Pad2) -> /Row_6
- D49 pad 2: Net-(D1-Pad2) -> /Row_1
- D5 pad 2: Net-(D11-Pad2) -> /Row_5
- D50 pad 2: Net-(D14-Pad2) -> /Row_2
- D51 pad 2: Net-(D15-Pad2) -> /Row_3
- D52 pad 2: Net-(D10-Pad2) -> /Row_4
- D53 pad 2: Net-(D11-Pad2) -> /Row_5
- D54 pad 2: Net-(D12-Pad2) -> /Row_6
- D55 pad 2: Net-(D1-Pad2) -> /Row_1
- D56 pad 2: Net-(D14-Pad2) -> /Row_2
- D57 pad 2: Net-(D15-Pad2) -> /Row_3
- D58 pad 2: Net-(D10-Pad2) -> /Row_4
- D59 pad 2: Net-(D11-Pad2) -> /Row_5
- D6 pad 2: Net-(D12-Pad2) -> /Row_6
- D60 pad 2: Net-(D12-Pad2) -> /Row_6
- D61 pad 2: Net-(D1-Pad2) -> /Row_1
- D62 pad 2: Net-(D14-Pad2) -> /Row_2
- D63 pad 2: Net-(D15-Pad2) -> /Row_3
- D64 pad 2: Net-(D10-Pad2) -> /Row_4
- D65 pad 2: Net-(D11-Pad2) -> /Row_5
- D66 pad 2: Net-(D12-Pad2) -> /Row_6
- D67 pad 2: Net-(D1-Pad2) -> /Row_1
- D68 pad 2: Net-(D14-Pad2) -> /Row_2
- D69 pad 2: Net-(D15-Pad2) -> /Row_3
- D7 pad 2: Net-(D1-Pad2) -> /Row_1
- D70 pad 2: Net-(D10-Pad2) -> /Row_4
- D71 pad 2: Net-(D11-Pad2) -> /Row_5
- D72 pad 2: Net-(D12-Pad2) -> /Row_6
- D73 pad 2: Net-(D1-Pad2) -> /Row_1
- D74 pad 2: Net-(D14-Pad2) -> /Row_2
- D75 pad 2: Net-(D15-Pad2) -> /Row_3
- D76 pad 2: Net-(D10-Pad2) -> /Row_4
- D77 pad 2: Net-(D11-Pad2) -> /Row_5
- D78 pad 2: Net-(D12-Pad2) -> /Row_6
- D79 pad 2: Net-(D1-Pad2) -> /Row_1
- D8 pad 2: Net-(D14-Pad2) -> /Row_2
- D80 pad 2: Net-(D14-Pad2) -> /Row_2
- D81 pad 2: Net-(D15-Pad2) -> /Row_3
- D82 pad 2: Net-(D10-Pad2) -> /Row_4
- D83 pad 2: Net-(D11-Pad2) -> /Row_5
- D84 pad 2: Net-(D12-Pad2) -> /Row_6
- D9 pad 2: Net-(D15-Pad2) -> /Row_3
- DOT1 pad 4: Net-(Bb1-Pad4) -> /LED_C3
- DOWN1 pad 1: Net-(D78-Pad1) -> Net-(D72-Pad1)
- DOWN1 pad 2: Net-(BACKSLASH1-Pad2) -> Net-(DOWN1-Pad2)
- DOWN1 pad 4: Net-(Bb1-Pad4) -> /LED_C3
- END1 pad 1: Net-(D83-Pad1) -> Net-(D85-Pad1)
- END1 pad 2: Net-(DELETE1-Pad2) -> Net-(DEC1-Pad2)
- END1 pad 4: Net-(Bb1-Pad4) -> /LED_C1
- EQUAL1 pad 4: Net-(BACKSPACE1-Pad4) -> /LED_C1
- ESC1 pad 4: Net-(BACKSPACE1-Pad4) -> /LED_C1
- F1 pad 4: Net-(BACKSPACE1-Pad4) -> /LED_C1
- F10 pad 4: Net-(BACKSPACE1-Pad4) -> /LED_C1
- F11 pad 4: Net-(BACKSPACE1-Pad4) -> /LED_C1
- F12 pad 4: Net-(BACKSPACE1-Pad4) -> /LED_C1
- F2 pad 4: Net-(BACKSPACE1-Pad4) -> /LED_C1
- F3 pad 4: Net-(BACKSPACE1-Pad4) -> /LED_C1
- F4 pad 4: Net-(BACKSPACE1-Pad4) -> /LED_C1
- F5 pad 4: Net-(BACKSPACE1-Pad4) -> /LED_C1
- F6 pad 4: Net-(BACKSPACE1-Pad4) -> /LED_C1
- F7 pad 4: Net-(BACKSPACE1-Pad4) -> /LED_C1
- F8 pad 4: Net-(BACKSPACE1-Pad4) -> /LED_C1
- F9 pad 4: Net-(BACKSPACE1-Pad4) -> /LED_C1
- FUNC1 pad 4: Net-(Bb1-Pad4) -> /LED_C3
- Ff1 pad 4: Net-(Bb1-Pad4) -> /LED_C3
- GRAVE1 pad 4: Net-(BACKSPACE1-Pad4) -> /LED_C1
- Gg1 pad 4: Net-(Bb1-Pad4) -> /LED_C3
- HOME1 pad 1: Net-(D80-Pad1) -> Net-(D79-Pad1)
- HOME1 pad 2: Net-(DELETE1-Pad2) -> Net-(HOME1-Pad2)
- HOME1 pad 4: Net-(BACKSPACE1-Pad4) -> /LED_C1
- Hh1 pad 4: Net-(Bb1-Pad4) -> /LED_C3
- Jj1 pad 4: Net-(Bb1-Pad4) -> /LED_C3
- LALT1 pad 4: Net-(Bb1-Pad4) -> /LED_C3
- LCTRL1 pad 4: Net-(Bb1-Pad4) -> /LED_C3
- LEFT1 pad 2: Net-(LEFT1-Pad2) -> Net-(DOWN1-Pad2)
- LEFT1 pad 4: Net-(Bb1-Pad4) -> /LED_C3
- LSHIFT1 pad 4: Net-(Bb1-Pad4) -> /LED_C3
- MCU1 pad 12: Net-(D1-Pad2) -> Net-(DEL1-Pad2)
- MCU1 pad 14: Net-(D15-Pad2) -> /Row_6
- MCU1 pad 2: Net-(F8-Pad2) -> Net-(COMMA1-Pad2)
- MCU1 pad 3: Net-(COMMA1-Pad2) -> Net-(DOT1-Pad2)
- MCU1 pad 39: Net-(MCU1-Pad39) -> Net-(F8-Pad2)
- MCU1 pad 4: Net-(DOT1-Pad2) -> Net-(EQUAL1-Pad2)
- MCU1 pad 42: Net-(D10-Pad2) -> /Row_1
- MCU1 pad 5: Net-(EQUAL1-Pad2) -> Net-(DOWN1-Pad2)
- MCU1 pad 6: Net-(LEFT1-Pad2) -> Net-(BACKSLASH1-Pad2)
- MCU1 pad 7: Net-(BACKSLASH1-Pad2) -> Net-(HOME1-Pad2)
- MINUS1 pad 4: Net-(BACKSPACE1-Pad4) -> /LED_C1
- Mm1 pad 4: Net-(Bb1-Pad4) -> /LED_C3
- Nn1 pad 4: Net-(Bb1-Pad4) -> /LED_C3
- ONE1 pad 4: Net-(BACKSPACE1-Pad4) -> /LED_C1
- P_jump_trans1 pad 1: Net-(Bb1-Pad4) -> /LED_C3
- P_jump_trans3 pad 1: Net-(BACKSPACE1-Pad4) -> /LED_C1
- QUOTE1 pad 2: Net-(LEFT1-Pad2) -> Net-(DOWN1-Pad2)
- R72 pad 2: Net-(R72-Pad2) -> Net-(DOWN1-Pad3)
- R78 pad 2: Net-(DOWN1-Pad3) -> Net-(R78-Pad2)
- R79 pad 2: Net-(DELETE1-Pad3) -> Net-(HOME1-Pad3)
- R80 pad 2: Net-(HOME1-Pad3) -> Net-(NUMLOCK1-Pad3)
- R83 pad 2: Net-(END1-Pad3) -> Net-(NO1-Pad3)
- R84 pad 2: Net-(R84-Pad2) -> Net-(NO0-Pad3)
- RBRAKET1 pad 2: Net-(LEFT1-Pad2) -> Net-(DOWN1-Pad2)
- RBRAKET1 pad 4: Net-(BACKSPACE1-Pad4) -> /LED_C1
- RIGHT1 pad 1: Net-(D84-Pad1) -> Net-(D78-Pad1)
- RIGHT1 pad 2: Net-(DELETE1-Pad2) -> Net-(BACKSLASH1-Pad2)
- RIGHT1 pad 3: Net-(R84-Pad2) -> Net-(R78-Pad2)
- RIGHT1 pad 4: Net-(Bb1-Pad4) -> /LED_C3
- RSHIFT1 pad 2: Net-(LEFT1-Pad2) -> Net-(DOWN1-Pad2)
- SEVEN7 pad 4: Net-(BACKSPACE1-Pad4) -> /LED_C1
- SIX6 pad 4: Net-(BACKSPACE1-Pad4) -> /LED_C1
- SLASH1 pad 4: Net-(Bb1-Pad4) -> /LED_C3
- SPACE1 pad 4: Net-(Bb1-Pad4) -> /LED_C3
- THREE3 pad 4: Net-(BACKSPACE1-Pad4) -> /LED_C1
- TWO2 pad 4: Net-(BACKSPACE1-Pad4) -> /LED_C1
- Transistor1 pad 2: Net-(Bb1-Pad4) -> /LED_C3
- Transistor3 pad 2: Net-(BACKSPACE1-Pad4) -> /LED_C1
- UP1 pad 4: Net-(Bb1-Pad4) -> /LED_C3
- Vv1 pad 4: Net-(Bb1-Pad4) -> /LED_C3
- Xx1 pad 4: Net-(Bb1-Pad4) -> /LED_C3
- Yy1 pad 4: Net-(Bb1-Pad4) -> /LED_C3
- ZERO0 pad 4: Net-(BACKSPACE1-Pad4) -> /LED_C1
- Zz1 pad 4: Net-(Bb1-Pad4) -> /LED_C3
- ext_1 pad 7: Net-(MCU1-Pad39) -> Net-(MCU1-Pad45)
Routing:
- net Net-(BACKSPACE1-Pad4): track 1182.1 -> 0.00 mm
- net /LED_C1: track 0.00 -> 1182.1 mm
- net Net-(Bb1-Pad4): track 1150.2 -> 0.00 mm
- net /LED_C3: track 0.00 -> 1150.2 mm
- net Net-(D14-Pad2): track 475.8 -> 0.00 mm
- net /Row_2: track 0.00 -> 475.8 mm
- net Net-(D12-Pad2): track 394.4 -> 0.00 mm
- net /Row_6: track 0.00 -> 394.4 mm
- net Net-(D1-Pad2): track 387.1 -> 0.00 mm
- net /Row_1: track 0.00 -> 387.1 mm
- net Net-(D11-Pad2): track 384.5 -> 0.00 mm
- net /Row_5: track 0.00 -> 384.5 mm
- net Net-(D10-Pad2): track 372.2 -> 0.00 mm
- net /Row_4: track 0.00 -> 372.2 mm
- net Net-(LEFT1-Pad2): track 139.1 -> 0.00 mm
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- removed copper zone on B.Cu, net Net-(MCU1-Pad46)
- removed copper zone on F.Cu, net Net-(MCU1-Pad49)

Commit message: align key
Parts:
- moved PAUSE1 183.9 mm to (317.2, 77.2), turned to 180 degrees
- moved PRSCREEN1 166.7 mm to (336.2, 77.2), turned to 180 degrees
- moved NO4 151.0 mm to (355.3, 134.4), turned to 180 degrees
- moved NUMLOCK1 141.4 mm to (355.3, 96.3), turned to 180 degrees
- moved NO7 134.9 mm to (355.3, 115.3), turned to 180 degrees
- moved No8 116.7 mm to (374.3, 115.3), turned to 180 degrees
- moved No5 112.1 mm to (374.3, 134.4), turned to 180 degrees
- moved NO0 102.3 mm to (374.3, 172.5), turned to 180 degrees
- moved No9 98.9 mm to (393.4, 115.3), turned to 180 degrees
- moved No6 93.4 mm to (393.4, 134.4), turned to 180 degrees
- moved No3 91.0 mm to (393.4, 153.4), turned to 180 degrees
- moved NO1 89.2 mm to (355.3, 153.4), turned to 180 degrees
- moved No2 86.3 mm to (374.3, 153.4), turned to 180 degrees
- moved INS1 85.8 mm to (393.4, 77.2), turned to 180 degrees
- moved DEV1 52.0 mm to (374.3, 96.3), turned to 180 degrees
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
Commit message: wiring led
Parts:
- R85, R86, R87, R88, R89, R90, R91, R92, R93, R94, R95, R96, R97, R98, R99: moved to B.Cu
- moved R97 272.6 mm to (407.7, 72.1)
- moved D98 258.8 mm to (403.9, 103.1), turned to 270 degrees
- moved R98 258.2 mm to (407.4, 91.2)
- moved D97 255.3 mm to (404.0, 84.1), turned to 270 degrees
- moved R91 253.2 mm to (388.5, 72.1)
- moved D92 247.3 mm to (385.0, 103.1), turned to 270 degrees
- moved D91 244.0 mm to (384.9, 84.1), turned to 270 degrees
- moved R99 239.5 mm to (407.6, 119.8)
- moved D99 238.6 mm to (404.0, 131.7), turned to 270 degrees
- moved R93 237.8 mm to (388.5, 110.2)
- moved R92 237.7 mm to (388.5, 91.2)
- moved D85 237.5 mm to (366.1, 84.1), turned to 270 degrees
- moved R85 237.3 mm to (369.3, 72.1)
- moved D96 237.3 mm to (403.9, 169.8), turned to 270 degrees
- moved R86 232.2 mm to (369.5, 91.2)
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Routing:
- net Net-(D15-Pad2): track 481.0 -> 0.00 mm
- net /Row_3: track 0.00 -> 411.7 mm
- net /LED_C2: track 825.7 -> 947.1 mm
- net Net-(DEC1-Pad2): track 0.00 -> 109.8 mm
- net Net-(HOME1-Pad2): track 0.00 -> 108.9 mm
- net Net-(INS1-Pad2): track 0.00 -> 108.6 mm
- net Net-(Bb1-Pad2): track 211.9 -> 110.0 mm
- net /LED_C3: track 1150.2 -> 1241.7 mm
- net /Row_5: track 384.5 -> 466.5 mm
- net Net-(BACKSLASH1-Pad2): track 209.2 -> 127.9 mm
- net /Row_2: track 475.8 -> 404.2 mm
- net /Row_6: track 394.4 -> 462.9 mm
- net Net-(DEL1-Pad2): track 0.00 -> 47.6 mm
- net /Row_4: track 372.2 -> 410.3 mm
- net /LED_C1: track 1182.1 -> 1219.6 mm
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Other:
- board size 320 x 140 mm -> 380 x 140 mm

Commit message: wring controller
Parts:
- R_trans1, R_trans2, R_trans3, Transistor1, Transistor2, Transistor3: moved to B.Cu
- moved Transistor3 23.2 mm to (79.3, 67.7)
- moved R_trans3 23.1 mm to (84.5, 67.7)
- moved P_jump_trans3 20.7 mm to (72.7, 66.4)
- moved Transistor2 18.3 mm to (79.3, 63.9)
- moved R_trans2 18.1 mm to (84.5, 63.9)
- moved P_jump_trans2 17.6 mm to (72.7, 63.9)
- moved Transistor1 15.9 mm to (79.3, 60.1)
- moved P_jump_trans1 15.7 mm to (72.7, 61.4)
- moved R_trans1 15.6 mm to (84.5, 60.1)
Connections:
- R_trans1 pad 2: Net-(MCU1-Pad26) -> Net-(MCU1-Pad24)
- R_trans3 pad 2: Net-(MCU1-Pad24) -> Net-(MCU1-Pad26)
Routing:
- net Net-(DEL1-Pad2): track 47.6 -> 363.3 mm
- net Net-(INS1-Pad2): track 108.6 -> 407.5 mm
- net Net-(DEC1-Pad2): track 109.8 -> 391.8 mm
- net Net-(HOME1-Pad2): track 108.9 -> 379.1 mm
- net Net-(BACKSLASH1-Pad2): track 127.9 -> 381.3 mm
- net Net-(DOWN1-Pad2): track 138.6 -> 374.8 mm
- net Net-(EQUAL1-Pad2): track 139.5 -> 370.6 mm
- net Net-(DOT1-Pad2): track 110.0 -> 313.3 mm
- net /Row_6: track 462.9 -> 658.6 mm, vias 0 -> 1
- net Net-(COMMA1-Pad2): track 110.0 -> 296.7 mm
- net /Row_5: track 466.5 -> 643.6 mm, vias 0 -> 1
- net /Row_4: track 410.3 -> 570.9 mm, vias 0 -> 1
- net /Row_2: track 404.2 -> 520.8 mm
- net Net-(F8-Pad2): track 109.1 -> 222.3 mm
- net Net-(Bb1-Pad2): track 110.0 -> 208.1 mm
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