File: main_board4.kicad_pcb (KiCad board)
At the start: 2 copper layers, 380 x 140 mm, 308 parts

Commit message: modify ext module
Parts:
- ext_1: footprint sw_fprint_wLed:ext_module_footprint -> sw_fprint_wLed:ext_module_footprint_v2
- moved ext_1 164.3 mm to (147.6, 110.5)
- moved R_trans1 14.5 mm to (98.7, 62.6), turned to 270 degrees
- moved R_trans2 11.8 mm to (96.2, 62.6), turned to 270 degrees
- moved R_trans3 10.5 mm to (93.7, 62.6), turned to 270 degrees
- moved Transistor3 7.67 mm to (86.9, 66.8)
- moved Transistor2 5.59 mm to (84.9, 63.8)
- moved P_jump_trans1 5.08 mm to (77.8, 61.4)
- moved P_jump_trans2 5.08 mm to (77.8, 63.9)
- moved P_jump_trans3 5.08 mm to (77.8, 66.4)
- moved Transistor1 3.61 mm to (82.9, 60.7)
- moved D4 2.92 mm to (64.2, 141.2)
Routing:
- net Net-(MCU1-Pad27): track 0.00 -> 140.7 mm
- net Net-(MCU1-Pad0): track 0.00 -> 89.3 mm
- net Net-(MCU1-Pad1): track 0.00 -> 87.8 mm
- net /Row_3: track 480.9 -> 562.1 mm
- net Net-(MCU1-Pad45): track 0.00 -> 44.0 mm
- net Net-(MCU1-Pad24): track 17.5 -> 3.23 mm
- net Net-(R_trans1-Pad1): track 3.21 -> 16.1 mm
- net /Row_1: track 449.9 -> 461.4 mm
- net /Row_2: track 520.8 -> 531.2 mm
- net Net-(R_trans2-Pad1): track 3.21 -> 13.2 mm
- net Net-(MCU1-Pad25): track 12.6 -> 3.23 mm
- net Net-(MCU1-Pad26): track 12.0 -> 3.25 mm
- net /LED_C1: track 1160.0 -> 1167.7 mm
- net Net-(R_trans3-Pad1): track 3.21 -> 10.9 mm
- net /LED_C2: track 941.1 -> 948.6 mm
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- added copper zone on B.Cu, net Net-(MCU1-Pad46)
- added copper zone on F.Cu, net Net-(MCU1-Pad49)

Commit message: working on trans
Parts:
- moved Transistor3 11.8 mm to (75.2, 66.7), turned to 90 degrees
- moved P_jump_trans1 11.4 mm to (66.3, 61.4)
- moved R_trans1 10.3 mm to (89.3, 58.4), turned to 0 degrees
- moved P_jump_trans2 9.25 mm to (68.9, 61.4)
- moved P_jump_trans3 8.13 mm to (71.4, 61.4)
- moved R_trans2 7.04 mm to (89.3, 61.2), turned to 0 degrees
- moved Transistor2 5.86 mm to (79.2, 62.3), turned to 90 degrees
- moved R_trans3 4.58 mm to (89.3, 64.0), turned to 0 degrees
- moved Transistor1 2.91 mm to (83.1, 57.8), turned to 90 degrees
Routing:
- net Net-(MCU1-Pad49): track 0.00 -> 15.5 mm
- net Net-(MCU1-Pad24): track 3.23 -> 16.1 mm
- net Net-(R_trans1-Pad1): track 16.1 -> 5.97 mm
- net Net-(MCU1-Pad25): track 3.23 -> 10.3 mm
- net /LED_C1: track 1167.7 -> 1162.1 mm
- net Net-(R_trans2-Pad1): track 13.2 -> 9.12 mm, vias 0 -> 2
- net Net-(R_trans3-Pad1): track 10.9 -> 13.9 mm, vias 0 -> 2
- net Net-(MCU1-Pad26): track 3.25 -> 5.41 mm
- net /LED_C3: track 1197.0 -> 1198.9 mm
- net /LED_C2: track 948.6 -> 947.9 mm
- net /Row_5: track 649.8 -> 649.3 mm
- added copper zone on F.Cu, net (none)
- removed copper zone on F.Cu, net Net-(MCU1-Pad49)
