File: main_board4.kicad_pcb (KiCad board)
At the start: 2 copper layers, 380 x 140 mm, 308 parts

Commit message: done
Parts:
- moved Transistor1 7.81 mm to (75.2, 57.8)
- moved D4 2.98 mm to (61.3, 140.3)
- moved Transistor3 2.21 mm to (75.2, 68.9)
Routing:
- net Net-(MCU1-Pad49): track 15.5 -> 122.6 mm, vias 0 -> 3
- net Net-(MCU1-Pad46): track 0.00 -> 12.3 mm, vias 0 -> 2
- net /Row_1: track 461.4 -> 453.3 mm
- net /Row_2: track 531.2 -> 523.3 mm
- net Net-(R_trans1-Pad1): track 5.97 -> 13.8 mm
- net /Row_3: track 562.1 -> 554.4 mm
- net /LED_C3: track 1198.9 -> 1194.6 mm
- net Net-(CAPLOCK1-Pad1): track 9.94 -> 13.2 mm
- net Net-(MCU1-Pad1): track 87.8 -> 86.0 mm
- net /LED_C2: track 947.9 -> 949.2 mm
- net /Row_4: track 575.4 -> 576.4 mm
- net Net-(R_trans3-Pad1): track 13.9 -> 14.8 mm

Commit message: align text
Parts:
- removed R_trans2: R, Resistor_SMD:R_0805_2012Metric
- added Rtrs2: R, Resistor_SMD:R_0805_2012Metric, B.Cu at (89.3, 61.2)
- PJT1: renamed from P_jump_trans1; value CONN_01X01 -> CON1
- PJT2: renamed from P_jump_trans2; value CONN_01X01 -> CON2
- PJT3: renamed from P_jump_trans3; value CONN_01X01 -> CON3
- renumbered Aa1 to Aa, BACKSLASH1 to BACKSLASH, BACKSPACE1 to BACKSPACE, Bb1 to Bb, CAPLOCK1 to CAPLOCK, RBRAKET1 to CBRAKET, COMMA1 to COMMA, COMMAND1 to COMMAND, Cc1 to Cc, MINUS1 to DASH, DEC1 to DEC, DEL1 to DELETE, DEV1 to DIV, DOT1 to DOT, DOWN1 to DOWN, Dd1 to Dd, END1 to END, ENTER1 to ENTER, EQUAL1 to EQUAL, ESC1 to ESC, Ee1 to Ee, FUNC1 to FUNC, Ff1 to Ff, GRAVE1 to GRAVE, Gg1 to Gg, HOME1 to HOME, Hh1 to Hh, INS1 to INSERT, Ii1 to Ii, Jj1 to Jj, Kk1 to Kk, LALT1 to LALT, LCTRL1 to LCTRL, LEFT1 to LEFT, LSHIFT1 to LSHIFT, Ll1 to Ll, MCU1 to MCU, MENU1 to MENU, R_minus1 to MINUS, MUL1 to MUL, Mm1 to Mm, No2 to NO2, No3 to NO3, No5 to NO5, No6 to NO6, No8 to NO8, No9 to NO9, NUMLOCK1 to NUMLOCK, Nn1 to Nn, LBRAKET1 to OBRAKET, Oo1 to Oo, PAUSE1 to PAUSE, PLUS1 to PLUS, PRSCREEN1 to PRSCREEN, Pp1 to Pp, QUOTE1 to QUOTE, Qq1 to Qq, RIGHT1 to RIGHT, RSHIFT1 to RSHIFT, Rr1 to Rr, R_trans1 to Rtrs1, R_trans3 to Rtrs3, SEMICOLON1 to SEMICOLON, SLASH1 to SLASH, SPACE1 to SPACE, Ss1 to Ss, TAB1 to TAB, Transistor1 to Trs1, Transistor2 to Trs2, Transistor3 to Trs3, Tt1 to Tt, UP1 to UP, Uu1 to Uu, R_Enter1 to V_ENTER, Vv1 to Vv, Ww1 to Ww, Xx1 to Xx, Yy1 to Yy, Zz1 to Zz

Commit message: adding mounthole
Parts:
- added REF**: Mounting_hole_M3, sw_fprint_wLed:Mounting_hole_M3, F.Cu at (56.0, 53.0)
- added REF**: Mounting_hole_M3, sw_fprint_wLed:Mounting_hole_M3, F.Cu at (420.0, 56.0)
- added REF**: Mounting_hole_M3, sw_fprint_wLed:Mounting_hole_M3, F.Cu at (422.0, 180.0)
- added REF**: Mounting_hole_M3, sw_fprint_wLed:Mounting_hole_M3, F.Cu at (56.0, 182.0)
- added REF**: Mounting_hole_M3, sw_fprint_wLed:Mounting_hole_M3, F.Cu at (234.0, 181.0)
- added REF**: Mounting_hole_M3, sw_fprint_wLed:Mounting_hole_M3, F.Cu at (226.0, 53.0)
- added REF**: Mounting_hole_M3, sw_fprint_wLed:Mounting_hole_M3, F.Cu at (147.0, 114.0)
- added REF**: Mounting_hole_M3, sw_fprint_wLed:Mounting_hole_M3, F.Cu at (319.8, 115.5)
- added REF**: Photo_resistor_hole, sw_fprint_wLed:Photo_resistor_hole, F.Cu at (196.0, 62.4)
Routing:
- net /LED_C2: track 949.2 -> 945.6 mm

Commit message: adjust mounting hole
Parts:
- removed REF**: Mounting_hole_M3, sw_fprint_wLed:Mounting_hole_M3
- added M3_BM: Mounting_hole_M3, sw_fprint_wLed:Mounting_hole_M3, F.Cu at (230.0, 182.0)
- moved M3_TM 24.0 mm to (250.0, 52.0)
- moved M3_MR 15.4 mm to (330.0, 127.0)
- moved M3_ML 13.3 mm to (150.0, 127.0)
- moved M3_TR 6.40 mm to (425.0, 52.0)
- moved M3_BR 3.61 mm to (425.0, 182.0)
- moved M3_TL 1.41 mm to (55.0, 52.0)
- moved M3_BL 1.00 mm to (55.0, 182.0)
- renumbered REF** to M3_BL, REF** to M3_BR, REF** to M3_ML, REF** to M3_MR, REF** to M3_TL, REF** to M3_TM, REF** to M3_TR, REF** to photo_r_hole
Routing:
- net Net-(BACKSLASH1-Pad2): track 383.6 -> 392.7 mm
- net /Row_5: track 649.3 -> 646.4 mm
- net /LED_C3: track 1194.6 -> 1192.0 mm
- net /LED_C2: track 945.6 -> 947.2 mm
- net /Row_6: track 665.4 -> 664.3 mm

Commit message: decoration
Parts:
- moved D28 2.51 mm to (144.5, 122.2)
- moved M3_ML 2.00 mm to (150.0, 125.0)
- moved M3_MR 2.00 mm to (330.0, 125.0)
Routing:
- net Net-(HOME1-Pad2): track 381.4 -> 373.0 mm
- net Net-(BACKSLASH1-Pad2): track 392.7 -> 384.5 mm
- net Net-(DOWN1-Pad2): track 377.1 -> 369.2 mm
- net Net-(EQUAL1-Pad2): track 373.0 -> 365.3 mm
- net Net-(DEL1-Pad2): track 364.6 -> 357.1 mm
- net Net-(DOT1-Pad2): track 315.6 -> 308.1 mm
- net Net-(INS1-Pad2): track 408.8 -> 401.6 mm
- net Net-(COMMA1-Pad2): track 299.0 -> 292.0 mm
- net Net-(DEC1-Pad2): track 393.2 -> 386.4 mm
- net /Row_4: track 576.4 -> 581.0 mm
- net Net-(F6-Pad2): track 181.8 -> 185.6 mm
- net Net-(D28-Pad1): track 5.72 -> 8.38 mm
- net /Row_3: track 554.4 -> 555.9 mm
- net /LED_C2: track 947.2 -> 948.4 mm
- net Net-(Cc1-Pad2): track 176.7 -> 176.0 mm
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