File: main_board4.kicad_pcb (KiCad board)
At the start: 2 copper layers, 380 x 140 mm, 317 parts, among them M3_BL Mounting_hole_M3, M3_BM Mounting_hole_M3, M3_BR Mounting_hole_M3, M3_ML Mounting_hole_M3, M3_MR Mounting_hole_M3, M3_TL Mounting_hole_M3, M3_TM Mounting_hole_M3, M3_TR Mounting_hole_M3

Commit message: export gerber
Routing:
- net Net-(Cc1-Pad2): track 176.0 -> 179.1 mm
- net Net-(F2-Pad2): track 140.2 -> 143.2 mm
- net /Row_3: track 555.9 -> 558.2 mm
- net /LED_C1: track 1162.1 -> 1163.7 mm
- net Net-(Aa1-Pad2): track 134.0 -> 135.3 mm
- net Net-(HOME1-Pad2): track 373.0 -> 371.8 mm
- net Net-(CAPLOCK1-Pad2): track 146.7 -> 147.8 mm
- net Net-(MCU1-Pad49): track 123.2 -> 122.4 mm
- net /Row_5: track 646.4 -> 645.7 mm
- net Net-(F4-Pad2): track 153.2 -> 153.7 mm
Other:
- net class Default: clearance 0.2 -> 0.3
- rule trace_clearance: 0.2 -> 0.3
- board text added: "HCM City - Nov 22, 2018. Where there's a will, there's a way!"
- board text added: "Layout99_v1.0"
